Commit message: Refactor DiffBot URDF with parameters and corrections

File: DiffBot Lab: diffbot.urdf.xacro (robot description, xacro)
@@ -1,66 +1,90 @@
 <?xml version="1.0"?>
 <robot name="diffbot" xmlns:xacro="http://www.ros.org/wiki/xacro">
-<!-- Base -->
- <link name="base_link">
-  <visual>
-    <geometry>
-      <box size="0.4 0.3 1"/>
-    </geometry>
-    <material name="gray">
-      <color rgba="0.6 0.6 0.6 1"/>
-    </material>
-  </visual>
-  <collision>
-   <geometry>
-      <box size="0.4 0.3 0.1"/>
-   </geometry>
-  </collision>
-  <inertia>
-    <mass value="5"/>
-  </inertia>
- </link>
-<!-- Left Wheel -->
- <link name="left_wheel">
-  <visual>
-   <geometry>
-     <cylinder lenghth="0.05" radius="0.05"/>
-   </geometry>
-  </visual>
- </link>
-<!-- Right Wheel -->
- <link name="right_wheel">
-  <visual>
-   <geometry>
-     <cylinder lenghth="0.05" radius="0.05"/>
-   </geometry>
-  </visual>
- </link>
-<!-- Wheel Joints-->
- <joint name="left_wheel_joint" type="continuous">
-  <parent link="base_link"/>
-  <child link="left_wheel"/>
-  <origin xyz="0 0.15 0" rpy="0 1.5707 0"/>
-  <axis xyz="0 1 0"/>
- </joint>
- <joint name="right_wheel_joint" type="continuous">
-  <parent link="base_link"/>
-  <child link="right_wheel"/>
-  <origin xyz="0 -0.15 0" rpy="0 1.5707 0"/>
-  <axis xyz="0 1 0"/>
- </joint>
-<!-- Gazebo -->
- <gazebo>
-  <plugin name="diff_drive" filename="libgazebo_ros_diff_drive.so">
-   <ros><namespace>/diffbot</namespace></ros>
-   <update_rate>30</update_rate>
-   <left_joint>left_wheel_joint</left_joint>
-   <right_joint>right_wheel_joint</right_joint>
-   <wheel_separation>0.3</wheel_separation>
-   <wheel_diameter>0.1</wheel_diameter>
-   <cmd_vel_topic>cmd_vel</cmd_vel_topic>
-   <odom_topic>odom</odom_topic>
-   <odom_frame>odom</odom_frame>
-   <base_frame>base_link</base_frame>
-  </plugin>
- </gazebo>
+  <!-- PARAMETERS -->
+  <xacro:property name="wheel_radius" value="0.05"/>
+  <xacro:property name="wheel_width" value="0.05"/>
+  <xacro:property name="wheel_sep" value="0.30"/>
+  <!-- BASE -->
+  <link name="base_link">
+    <visual>
+      <geometry>
+        <box size="0.4 0.3 0.1"/>
+      </geometry>
+      <material><color rgba="0.6 0.6 0.6 1"/></material>
+    </visual>
+    <collision>
+      <geometry>
+        <box size="0.4 0.3 0.1"/>
+      </geometry>
+    </collision>
+    <inertial>
+      <mass value="5.0"/>
+      <inertia ixx="0.1" iyy="0.1" izz="0.1" ixy="0" ixz="0" iyz="0"/>
+    </inertial>
+  </link>
+  <!-- LEFT WHEEL -->
+  <link name="left_wheel">
+    <visual>
+      <geometry>
+        <cylinder radius="${wheel_radius}" length="${wheel_width}"/>
+      </geometry>
+      <material><color rgba="0 0 0 1"/></material>
+    </visual>
+    <collision>
+      <geometry>
+        <cylinder radius="${wheel_radius}" length="${wheel_width}"/>
+      </geometry>
+    </collision>
+    <inertial>
+      <mass value="1.0"/>
+      <inertia ixx="0.01" iyy="0.01" izz="0.01" ixy="0" ixz="0" iyz="0"/>
+    </inertial>
+  </link>
+  <!-- RIGHT WHEEL -->
+  <link name="right_wheel">
+    <visual>
+      <geometry>
+        <cylinder radius="${wheel_radius}" length="${wheel_width}"/>
+      </geometry>
+      <material><color rgba="0 0 0 1"/></material>
+    </visual>
+    <collision>
+      <geometry>
+        <cylinder radius="${wheel_radius}" length="${wheel_width}"/>
+      </geometry>
+    </collision>
+    <inertial>
+      <mass value="1.0"/>
+      <inertia ixx="0.01" iyy="0.01" izz="0.01" ixy="0" ixz="0" iyz="0"/>
+    </inertial>
+  </link>
+  <!-- LEFT JOINT -->
+  <joint name="left_wheel_joint" type="continuous">
+    <parent link="base_link"/>
+    <child link="left_wheel"/>
+    <origin xyz="0 ${wheel_sep/2} -0.05" rpy="0 1.5707 0"/>
+    <axis xyz="0 1 0"/>
+  </joint>
+  <!-- RIGHT JOINT -->
+  <joint name="right_wheel_joint" type="continuous">
+    <parent link="base_link"/>
+    <child link="right_wheel"/>
+    <origin xyz="0 -${wheel_sep/2} -0.05" rpy="0 1.5707 0"/>
+    <axis xyz="0 1 0"/>
+  </joint>
+  <!-- GAZEBO -->
+  <gazebo>
+    <plugin
+      filename="libros_gz_sim_diff_drive_system.so"
+      name="ros_diff_drive">
+      <left_joint>left_wheel_joint</left_joint>
+      <right_joint>right_wheel_joint</right_joint>
+      <wheel_separation>${wheel_sep}</wheel_separation>
+      <wheel_radius>${wheel_radius}</wheel_radius>
+      <command_topic>cmd_vel</command_topic>
+      <odom_topic>odom</odom_topic>
+      <odometry_frame>odom</odometry_frame>
+      <robot_base_frame>base_link</robot_base_frame>
+    </plugin>
+  </gazebo>
 </robot>

Commit message: Refactor DiffBot URDF for clarity and structure

File: DiffBot Lab: diffbot.urdf.xacro (robot description, xacro)
@@ -6,5 +6,7 @@
   <xacro:property name="wheel_width" value="0.05"/>
   <xacro:property name="wheel_sep" value="0.30"/>
-  <!-- BASE -->
+  <!-- Derived parameters -->
+  <xacro:property name="half_wheel_sep" value="${wheel_sep * 0.5}"/>
+  <!-- ================= BASE ================= -->
   <link name="base_link">
     <visual>
@@ -12,5 +14,7 @@
         <box size="0.4 0.3 0.1"/>
       </geometry>
-      <material><color rgba="0.6 0.6 0.6 1"/></material>
+      <material name="gray">
+        <color rgba="0.6 0.6 0.6 1"/>
+      </material>
     </visual>
     <collision>
@@ -21,8 +25,10 @@
     <inertial>
       <mass value="5.0"/>
-      <inertia ixx="0.1" iyy="0.1" izz="0.1" ixy="0" ixz="0" iyz="0"/>
+      <inertia
+        ixx="0.1" iyy="0.1" izz="0.1"
+        ixy="0.0" ixz="0.0" iyz="0.0"/>
     </inertial>
   </link>
-  <!-- LEFT WHEEL -->
+  <!-- ================= LEFT WHEEL ================= -->
   <link name="left_wheel">
     <visual>
@@ -30,5 +36,7 @@
         <cylinder radius="${wheel_radius}" length="${wheel_width}"/>
       </geometry>
-      <material><color rgba="0 0 0 1"/></material>
+      <material name="black">
+        <color rgba="0 0 0 1"/>
+      </material>
     </visual>
     <collision>
@@ -39,8 +47,10 @@
     <inertial>
       <mass value="1.0"/>
-      <inertia ixx="0.01" iyy="0.01" izz="0.01" ixy="0" ixz="0" iyz="0"/>
+      <inertia
+        ixx="0.01" iyy="0.01" izz="0.01"
+        ixy="0.0" ixz="0.0" iyz="0.0"/>
     </inertial>
   </link>
-  <!-- RIGHT WHEEL -->
+  <!-- ================= RIGHT WHEEL ================= -->
   <link name="right_wheel">
     <visual>
@@ -48,5 +58,7 @@
         <cylinder radius="${wheel_radius}" length="${wheel_width}"/>
       </geometry>
-      <material><color rgba="0 0 0 1"/></material>
+      <material name="black">
+        <color rgba="0 0 0 1"/>
+      </material>
     </visual>
     <collision>
@@ -57,22 +69,24 @@
     <inertial>
       <mass value="1.0"/>
-      <inertia ixx="0.01" iyy="0.01" izz="0.01" ixy="0" ixz="0" iyz="0"/>
+      <inertia
+        ixx="0.01" iyy="0.01" izz="0.01"
+        ixy="0.0" ixz="0.0" iyz="0.0"/>
     </inertial>
   </link>
-  <!-- LEFT JOINT -->
+  <!-- ================= LEFT JOINT ================= -->
   <joint name="left_wheel_joint" type="continuous">
     <parent link="base_link"/>
     <child link="left_wheel"/>
-    <origin xyz="0 ${wheel_sep/2} -0.05" rpy="0 1.5707 0"/>
+    <origin xyz="0 ${half_wheel_sep} -0.05" rpy="0 1.5707 0"/>
     <axis xyz="0 1 0"/>
   </joint>
-  <!-- RIGHT JOINT -->
+  <!-- ================= RIGHT JOINT ================= -->
   <joint name="right_wheel_joint" type="continuous">
     <parent link="base_link"/>
     <child link="right_wheel"/>
-    <origin xyz="0 -${wheel_sep/2} -0.05" rpy="0 1.5707 0"/>
+    <origin xyz="0 -${half_wheel_sep} -0.05" rpy="0 1.5707 0"/>
     <axis xyz="0 1 0"/>
   </joint>
-  <!-- GAZEBO -->
+  <!-- ================= GAZEBO DIFF DRIVE ================= -->
   <gazebo>
     <plugin

Commit message: Update DiffBot parameters and dimensions

File: DiffBot Lab: diffbot.urdf.xacro (robot description, xacro)
@@ -2,8 +2,8 @@
 <!-- CMP 438: Communicating Robots - Isaac D. Hoyos -->
 <robot name="diffbot" xmlns:xacro="http://www.ros.org/wiki/xacro">
-  <!-- PARAMETERS -->
-  <xacro:property name="wheel_radius" value="0.05"/>
-  <xacro:property name="wheel_width" value="0.05"/>
-  <xacro:property name="wheel_sep" value="0.30"/>
+  <!-- ================= PARAMETERS ================= -->
+  <xacro:property name="wheel_radius" value="0.075"/>
+  <xacro:property name="wheel_width" value="0.075"/>
+  <xacro:property name="wheel_sep" value="0.45"/>
   <!-- Derived parameters -->
   <xacro:property name="half_wheel_sep" value="${wheel_sep * 0.5}"/>
@@ -12,19 +12,20 @@
     <visual>
       <geometry>
-        <box size="0.4 0.3 0.1"/>
+        <!-- Bigger body -->
+        <box size="0.6 0.45 0.15"/>
       </geometry>
-      <material name="gray">
-        <color rgba="0.6 0.6 0.6 1"/>
+      <material name="green">
+        <color rgba="0 1 0 1"/>
       </material>
     </visual>
     <collision>
       <geometry>
-        <box size="0.4 0.3 0.1"/>
+        <box size="0.6 0.45 0.15"/>
       </geometry>
     </collision>
     <inertial>
-      <mass value="5.0"/>
+      <mass value="8.0"/>
       <inertia
-        ixx="0.1" iyy="0.1" izz="0.1"
+        ixx="0.2" iyy="0.2" izz="0.2"
         ixy="0.0" ixz="0.0" iyz="0.0"/>
     </inertial>
@@ -36,6 +37,6 @@
         <cylinder radius="${wheel_radius}" length="${wheel_width}"/>
       </geometry>
-      <material name="black">
-        <color rgba="0 0 0 1"/>
+      <material name="blue">
+        <color rgba="0 0 1 1"/>
       </material>
     </visual>
@@ -46,7 +47,7 @@
     </collision>
     <inertial>
-      <mass value="1.0"/>
+      <mass value="1.5"/>
       <inertia
-        ixx="0.01" iyy="0.01" izz="0.01"
+        ixx="0.02" iyy="0.02" izz="0.02"
         ixy="0.0" ixz="0.0" iyz="0.0"/>
     </inertial>
@@ -58,6 +59,6 @@
         <cylinder radius="${wheel_radius}" length="${wheel_width}"/>
       </geometry>
-      <material name="black">
-        <color rgba="0 0 0 1"/>
+      <material name="blue">
+        <color rgba="0 0 1 1"/>
       </material>
     </visual>
@@ -68,7 +69,7 @@
     </collision>
     <inertial>
-      <mass value="1.0"/>
+      <mass value="1.5"/>
       <inertia
-        ixx="0.01" iyy="0.01" izz="0.01"
+        ixx="0.02" iyy="0.02" izz="0.02"
         ixy="0.0" ixz="0.0" iyz="0.0"/>
     </inertial>
@@ -78,5 +79,5 @@
     <parent link="base_link"/>
     <child link="left_wheel"/>
-    <origin xyz="0 ${half_wheel_sep} -0.05" rpy="0 1.5707 0"/>
+    <origin xyz="0 ${half_wheel_sep} -0.075" rpy="0 1.5707 0"/>
     <axis xyz="0 1 0"/>
   </joint>
@@ -85,5 +86,5 @@
     <parent link="base_link"/>
     <child link="right_wheel"/>
-    <origin xyz="0 -${half_wheel_sep} -0.05" rpy="0 1.5707 0"/>
+    <origin xyz="0 -${half_wheel_sep} -0.075" rpy="0 1.5707 0"/>
     <axis xyz="0 1 0"/>
   </joint>

Commit message: Update DiffBot URDF parameters and structure

File: DiffBot Lab: diffbot.urdf.xacro (robot description, xacro)
@@ -3,13 +3,14 @@
 <robot name="diffbot" xmlns:xacro="http://www.ros.org/wiki/xacro">
   <!-- ================= PARAMETERS ================= -->
-  <xacro:property name="wheel_radius" value="0.075"/>
-  <xacro:property name="wheel_width" value="0.075"/>
-  <xacro:property name="wheel_sep" value="0.45"/>
+  <xacro:property name="wheel_radius" value="0.05"/>
+  <xacro:property name="wheel_width" value="0.05"/>
+  <xacro:property name="wheel_sep" value="0.30"/>
   <xacro:property name="half_wheel_sep" value="${wheel_sep * 0.5}"/>
-  <!-- ================= BASE ================= -->
-  <link name="base_link">
+  <!-- ================= BASE BODY ================= -->
+  <link name="base_link"/>
+  <link name="base_body">
     <visual>
       <geometry>
-        <box size="0.6 0.45 0.15"/>
+        <box size="0.4 0.3 0.1"/>
       </geometry>
       <material name="green">
@@ -19,14 +20,19 @@
     <collision>
       <geometry>
-        <box size="0.6 0.45 0.15"/>
+        <box size="0.4 0.3 0.1"/>
       </geometry>
     </collision>
     <inertial>
-      <mass value="8.0"/>
+      <mass value="5.0"/>
       <inertia
-        ixx="0.2" iyy="0.2" izz="0.2"
+        ixx="0.1" iyy="0.1" izz="0.1"
         ixy="0.0" ixz="0.0" iyz="0.0"/>
     </inertial>
   </link>
+  <joint name="base_body_joint" type="fixed">
+    <parent link="base_link"/>
+    <child link="base_body"/>
+    <origin xyz="0 0 0.10" rpy="0 0 0"/>
+  </joint>
   <!-- ================= LEFT WHEEL ================= -->
   <link name="left_wheel">
@@ -45,7 +51,7 @@
     </collision>
     <inertial>
-      <mass value="1.5"/>
+      <mass value="1.0"/>
       <inertia
-        ixx="0.02" iyy="0.02" izz="0.02"
+        ixx="0.01" iyy="0.01" izz="0.01"
         ixy="0.0" ixz="0.0" iyz="0.0"/>
     </inertial>
@@ -67,22 +73,21 @@
     </collision>
     <inertial>
-      <mass value="1.5"/>
+      <mass value="1.0"/>
       <inertia
-        ixx="0.02" iyy="0.02" izz="0.02"
+        ixx="0.01" iyy="0.01" izz="0.01"
         ixy="0.0" ixz="0.0" iyz="0.0"/>
     </inertial>
   </link>
-  <!-- ================= LEFT JOINT ================= -->
+  <!-- ================= WHEEL JOINTS ================= -->
   <joint name="left_wheel_joint" type="continuous">
     <parent link="base_link"/>
     <child link="left_wheel"/>
-    <origin xyz="0 ${half_wheel_sep} -0.075" rpy="0 1.5707 0"/>
+    <origin xyz="0 ${half_wheel_sep} 0.05" rpy="0 1.5707 0"/>
     <axis xyz="0 1 0"/>
   </joint>
-  <!-- ================= RIGHT JOINT ================= -->
   <joint name="right_wheel_joint" type="continuous">
     <parent link="base_link"/>
     <child link="right_wheel"/>
-    <origin xyz="0 -${half_wheel_sep} -0.075" rpy="0 1.5707 0"/>
+    <origin xyz="0 -${half_wheel_sep} 0.05" rpy="0 1.5707 0"/>
     <axis xyz="0 1 0"/>
   </joint>
